Commit message: replaced 'basic_robot' with 'fus_bot'

File: urdf/fus_bot.xacro (robot description, xacro)
@@ -1,7 +1,7 @@
 <?xml version="1.0" ?>
-<robot name="Basic_Robot" xmlns:xacro="http://www.ros.org/wiki/xacro">
-<xacro:include filename="$(find Basic_Robot_description)/urdf/materials.xacro" />
-<xacro:include filename="$(find Basic_Robot_description)/urdf/Basic_Robot.trans" />
-<xacro:include filename="$(find Basic_Robot_description)/urdf/Basic_Robot.gazebo" />
+<robot name="fus_bot" xmlns:xacro="http://www.ros.org/wiki/xacro">
+<xacro:include filename="$(find fus_bot_description)/urdf/materials.xacro" />
+<xacro:include filename="$(find fus_bot_description)/urdf/fus_bot.trans" />
+<xacro:include filename="$(find fus_bot_description)/urdf/fus_bot.gazebo" />
 <link name="base_link">
   <inertial>
@@ -13,5 +13,5 @@
     <origin rpy="0 0 0" xyz="0 0 0"/>
     <geometry>
-      <mesh filename="package://Basic_Robot_description/meshes/base_link.stl" scale="0.001 0.001 0.001"/>
+      <mesh filename="package://fus_bot_description/meshes/base_link.stl" scale="0.001 0.001 0.001"/>
     </geometry>
     <material name="silver"/>
@@ -20,5 +20,5 @@
     <origin rpy="0 0 0" xyz="0 0 0"/>
     <geometry>
-      <mesh filename="package://Basic_Robot_description/meshes/base_link.stl" scale="0.001 0.001 0.001"/>
+      <mesh filename="package://fus_bot_description/meshes/base_link.stl" scale="0.001 0.001 0.001"/>
     </geometry>
   </collision>
@@ -33,5 +33,5 @@
     <origin rpy="0 0 0" xyz="-0.0 -0.005 0.06"/>
     <geometry>
-      <mesh filename="package://Basic_Robot_description/meshes/right_wheel_1.stl" scale="0.001 0.001 0.001"/>
+      <mesh filename="package://fus_bot_description/meshes/right_wheel_1.stl" scale="0.001 0.001 0.001"/>
     </geometry>
     <material name="silver"/>
@@ -40,5 +40,5 @@
     <origin rpy="0 0 0" xyz="-0.0 -0.005 0.06"/>
     <geometry>
-      <mesh filename="package://Basic_Robot_description/meshes/right_wheel_1.stl" scale="0.001 0.001 0.001"/>
+      <mesh filename="package://fus_bot_description/meshes/right_wheel_1.stl" scale="0.001 0.001 0.001"/>
     </geometry>
   </collision>
@@ -53,5 +53,5 @@
     <origin rpy="0 0 0" xyz="-0.0 -0.005 -0.0"/>
     <geometry>
-      <mesh filename="package://Basic_Robot_description/meshes/left_wheel_1.stl" scale="0.001 0.001 0.001"/>
+      <mesh filename="package://fus_bot_description/meshes/left_wheel_1.stl" scale="0.001 0.001 0.001"/>
     </geometry>
     <material name="silver"/>
@@ -60,5 +60,5 @@
     <origin rpy="0 0 0" xyz="-0.0 -0.005 -0.0"/>
     <geometry>
-      <mesh filename="package://Basic_Robot_description/meshes/left_wheel_1.stl" scale="0.001 0.001 0.001"/>
+      <mesh filename="package://fus_bot_description/meshes/left_wheel_1.stl" scale="0.001 0.001 0.001"/>
     </geometry>
   </collision>

Commit message: fixed previous naming overlooked _description suffix and added dummy link

File: urdf/fus_bot.xacro (robot description, xacro)
@@ -1,7 +1,9 @@
 <?xml version="1.0" ?>
 <robot name="fus_bot" xmlns:xacro="http://www.ros.org/wiki/xacro">
-<xacro:include filename="$(find fus_bot_description)/urdf/materials.xacro" />
-<xacro:include filename="$(find fus_bot_description)/urdf/fus_bot.trans" />
-<xacro:include filename="$(find fus_bot_description)/urdf/fus_bot.gazebo" />
+<xacro:include filename="$(find fus_bot)/urdf/materials.xacro" />
+<xacro:include filename="$(find fus_bot)/urdf/fus_bot.trans" />
+<xacro:include filename="$(find fus_bot)/urdf/fus_bot.gazebo" />
+<link name="dummy">
+</link>
 <link name="base_link">
   <inertial>
@@ -13,5 +15,5 @@
     <origin rpy="0 0 0" xyz="0 0 0"/>
     <geometry>
-      <mesh filename="package://fus_bot_description/meshes/base_link.stl" scale="0.001 0.001 0.001"/>
+      <mesh filename="package://fus_bot/meshes/base_link.stl" scale="0.001 0.001 0.001"/>
     </geometry>
     <material name="silver"/>
@@ -20,5 +22,5 @@
     <origin rpy="0 0 0" xyz="0 0 0"/>
     <geometry>
-      <mesh filename="package://fus_bot_description/meshes/base_link.stl" scale="0.001 0.001 0.001"/>
+      <mesh filename="package://fus_bot/meshes/base_link.stl" scale="0.001 0.001 0.001"/>
     </geometry>
   </collision>
@@ -33,5 +35,5 @@
     <origin rpy="0 0 0" xyz="-0.0 -0.005 0.06"/>
     <geometry>
-      <mesh filename="package://fus_bot_description/meshes/right_wheel_1.stl" scale="0.001 0.001 0.001"/>
+      <mesh filename="package://fus_bot/meshes/right_wheel_1.stl" scale="0.001 0.001 0.001"/>
     </geometry>
     <material name="silver"/>
@@ -40,5 +42,5 @@
     <origin rpy="0 0 0" xyz="-0.0 -0.005 0.06"/>
     <geometry>
-      <mesh filename="package://fus_bot_description/meshes/right_wheel_1.stl" scale="0.001 0.001 0.001"/>
+      <mesh filename="package://fus_bot/meshes/right_wheel_1.stl" scale="0.001 0.001 0.001"/>
     </geometry>
   </collision>
@@ -53,5 +55,5 @@
     <origin rpy="0 0 0" xyz="-0.0 -0.005 -0.0"/>
     <geometry>
-      <mesh filename="package://fus_bot_description/meshes/left_wheel_1.stl" scale="0.001 0.001 0.001"/>
+      <mesh filename="package://fus_bot/meshes/left_wheel_1.stl" scale="0.001 0.001 0.001"/>
     </geometry>
     <material name="silver"/>
@@ -60,8 +62,12 @@
     <origin rpy="0 0 0" xyz="-0.0 -0.005 -0.0"/>
     <geometry>
-      <mesh filename="package://fus_bot_description/meshes/left_wheel_1.stl" scale="0.001 0.001 0.001"/>
+      <mesh filename="package://fus_bot/meshes/left_wheel_1.stl" scale="0.001 0.001 0.001"/>
     </geometry>
   </collision>
 </link>
+<joint name="dummy_joint" type="fixed">
+  <parent link="dummy"/>
+  <child link="base_link"/>
+</joint>
 <joint name="Rev1" type="continuous">
   <origin rpy="0 0 0" xyz="0.0 0.005 -0.06"/>
